Commit message: Fix link inertials and add DYNAMIXEL actuator config
Inertials (verified against mesh-derived COM/inertia for all links):
- foot: tensor entries were misplaced (negative izz, not positive-definite)
- ankle_roll_pitch: COM missing the visual origin offset
- back_thigh/back_shin: inconsistent copied mass/inertia; mass from Al density
- elbow_yaw/elbow_pitch/gripper: CAD values re-expressed in the link frame
  (visuals are rotated +-90 deg; COM was off by 42-66 mm)
- lower_body/upper_body/shoulder/head: products of inertia sign flipped to
  URDF convention; lower_body COM missing visual z offset
- knee/front_thigh/front_shin: replaced hand-entered tensors with mesh values

Actuators:
- config/actuators.yaml: single source for XH540-W270, XM540-W270,
  XM430-W350 specs at 14.8 V, joint-to-servo mapping (dual servos on hip
  pitch and knee), armature/friction priors transferred from BAM MX-series
  identifications, and BAM identification priors
- urdf/actuators.xacro: generates joint <limit>/<dynamics> from the yaml
- hip_yaw now uses XM540-W270 limits (was XM430 values)
- left_front_thigh effort fixed to dual-servo value
- Install config/ in setup.py; regenerate robinion2.urdf

File: urdf/body.xacro (robot description, xacro)
@@ -22,9 +22,9 @@
       </collision>
       <inertial>
-        <origin xyz="-0.007122 0.000256 0.034914" rpy="0.0 0.0 0.0"/>
+        <origin xyz="-0.007122 0.000256 0.040914" rpy="0.0 0.0 0.0"/>
         <mass value="0.960747"/>
         <inertia
-          ixx="0.002662" ixy="0.000002" ixz="0.000113"
-          iyy="0.001197" iyz="0.000003"
+          ixx="0.002662" ixy="-0.000002" ixz="-0.000113"
+          iyy="0.001197" iyz="-0.000003"
           izz="0.002578"/>
       </inertial>
@@ -35,6 +35,5 @@
       <origin xyz="0.019 0.0245 0.07675" rpy="0.0 0.0 0.0"/>
       <axis xyz="0 1 0"/>
-      <limit velocity="3.14" effort="10.6" lower="-0.52" upper="${pi*0.5}"/>
-      <dynamics damping="0.1" friction="0.0"/>
+      <xacro:dxl_joint_props joint="torso_pitch_joint" lower="-0.52" upper="${pi*0.5}"/>
     </joint>
     <link name="upper_body_link">
@@ -55,6 +54,6 @@
         <mass value="1.234139"/>
         <inertia
-          ixx="0.006795" ixy="0.000000" ixz="-0.000098"
-          iyy="0.003101" iyz="-0.000005"
+          ixx="0.006795" ixy="0.000000" ixz="0.000098"
+          iyy="0.003101" iyz="0.000005"
           izz="0.006100"/>
       </inertial>

File: urdf/head.xacro (robot description, xacro)
@@ -7,6 +7,5 @@
       <origin xyz="-0.0125 -0.0245 0.183051" rpy="0.0 0.0 0.0"/>
       <axis xyz="0 0 1"/>
-      <limit velocity="4.82" effort="4.1" lower="${-pi*0.5}" upper="${pi*0.5}"/>
-      <dynamics damping="0.1" friction="0.0"/>
+      <xacro:dxl_joint_props joint="head_yaw_joint" lower="${-pi*0.5}" upper="${pi*0.5}"/>
     </joint>
     <link name="head_yaw_link">
@@ -31,6 +30,5 @@
       <origin xyz="0.000 0.019 0.047" rpy="0.0 0.0 0.0"/>
       <axis xyz="0 -1 0"/>
-      <limit velocity="4.82" effort="4.1" lower="${-pi*0.5}" upper="${pi*0.5}"/>
-      <dynamics damping="0.1" friction="0.0"/>
+      <xacro:dxl_joint_props joint="head_pitch_joint" lower="${-pi*0.5}" upper="${pi*0.5}"/>
     </joint>
     <link name="head_pitch_link">
@@ -51,6 +49,6 @@
         <mass value="0.164500"/>
         <inertia
-          ixx="0.000115" ixy="0.000000" ixz="0.000005"
-          iyy="0.000092" iyz="0.000001"
+          ixx="0.000115" ixy="0.000000" ixz="-0.000005"
+          iyy="0.000092" iyz="-0.000001"
           izz="0.000047"/>
       </inertial>

File: urdf/left_arm.xacro (robot description, xacro)
@@ -7,6 +7,5 @@
       <origin xyz="-0.02089 0.0815 0.1388" rpy="0 0.0873 0"/>
       <axis xyz="0 1 0"/>
-      <limit velocity="3.14" effort="10.6" lower="${-pi*0.9}" upper="${pi*0.9}"/>
-      <dynamics damping="0.1" friction="0.0"/>
+      <xacro:dxl_joint_props joint="left_shoulder_pitch_joint" lower="${-pi*0.9}" upper="${pi*0.9}"/>
     </joint>
     <link name="left_shoulder_pitch_link">
@@ -22,5 +21,5 @@
         <inertia
           ixx="0.000013" ixy="0.000000" ixz="0.000000"
-          iyy="0.000027" iyz="-0.000003"
+          iyy="0.000027" iyz="0.000003"
           izz="0.000025"/>
       </inertial>
@@ -31,6 +30,5 @@
       <origin xyz="0.0245 0.030017 -0.022" rpy="0.0 0.0 0.0"/>
       <axis xyz="1 0 0"/>
-      <limit velocity="3.14" effort="10.6" lower="${-pi*0.5}" upper="${pi*0.5}"/>
-      <dynamics damping="0.1" friction="0.0"/>
+      <xacro:dxl_joint_props joint="left_shoulder_roll_joint" lower="${-pi*0.5}" upper="${pi*0.5}"/>
     </joint>
     <link name="left_shoulder_roll_link">
@@ -51,5 +49,5 @@
         <mass value="0.389041"/>
         <inertia
-          ixx="0.000698" ixy="-0.000079" ixz="0.000000"
+          ixx="0.000698" ixy="0.000079" ixz="0.000000"
           iyy="0.000117" iyz="0.000000"
           izz="0.000753"/>
@@ -61,6 +59,5 @@
       <origin xyz="-0.0245 0.118 0.000" rpy="${pi*0.5} 0.0 0.0"/>
       <axis xyz="0 0 1"/>
-      <limit velocity="4.82" effort="4.1" lower="${-pi*0.9}" upper="${pi*0.9}"/>
-      <dynamics damping="0.1" friction="0.0"/>
+      <xacro:dxl_joint_props joint="left_elbow_yaw_joint" lower="${-pi*0.9}" upper="${pi*0.9}"/>
     </joint>
     <link name="left_elbow_yaw_link">
@@ -72,10 +69,10 @@
       </visual>
       <inertial>
-        <origin xyz="0.003756 0.032656 0.000000" rpy="0.0 0.0 0.0"/>
+        <origin xyz="0.003756 0.000000 -0.032656" rpy="0.0 0.0 0.0"/>
         <mass value="0.051730"/>
         <inertia
-          ixx="0.000036" ixy="0.000005" ixz="0.000000"
-          iyy="0.000028" iyz="0.000000"
-          izz="0.000025"/>
+          ixx="0.000036" ixy="0.000000" ixz="0.000005"
+          iyy="0.000025" iyz="0.000000"
+          izz="0.000028"/>
       </inertial>
     </link>
@@ -85,6 +82,5 @@
       <origin xyz="0.022 0.0245 -0.06" rpy="0.0 0.0 0.0"/>
       <axis xyz="0 1 0"/>
-      <limit velocity="3.14" effort="10.6" lower="${-pi*0.5}" upper="${pi*0.5}"/>
-      <dynamics damping="0.1" friction="0.0"/>
+      <xacro:dxl_joint_props joint="left_elbow_pitch_joint" lower="${-pi*0.5}" upper="${pi*0.5}"/>
     </joint>
     <link name="left_elbow_pitch_link">
@@ -102,10 +98,10 @@
       </collision>
       <inertial>
-        <origin xyz="0.000000 0.018081 -0.023869" rpy="0.0 0.0 0.0"/>
+        <origin xyz="0.000000 -0.023869 -0.018081" rpy="0.0 0.0 0.0"/>
         <mass value="0.246669"/>
         <inertia
           ixx="0.000135" ixy="0.000000" ixz="0.000000"
-          iyy="0.000064" iyz="-0.000001"
-          izz="0.000121"/>
+          iyy="0.000121" iyz="-0.000001"
+          izz="0.000064"/>
       </inertial>
     </link>
@@ -129,10 +125,10 @@
       </collision>
       <inertial>
-        <origin xyz="0.000002 0.043774 0.003217" rpy="0.0 0.0 0.0"/>
+        <origin xyz="0.000002 0.003217 -0.043774" rpy="0.0 0.0 0.0"/>
         <mass value="0.216195"/>
         <inertia
           ixx="0.000183" ixy="0.000000" ixz="0.000000"
-          iyy="0.000104" iyz="0.000015"
-          izz="0.000191"/>
+          iyy="0.000191" iyz="0.000015"
+          izz="0.000104"/>
       </inertial>
     </link>

File: urdf/left_leg.xacro (robot description, xacro)
@@ -7,6 +7,5 @@
       <origin xyz="0.0 0.055 0.0" rpy="0.0 0.0 0.0"/>
       <axis xyz="0 0 1"/>
-      <limit velocity="4.82" effort="4.1" lower="${-pi*0.5}" upper="${pi*0.5}"/>
-      <dynamics damping="0.1" friction="0.0"/>
+      <xacro:dxl_joint_props joint="left_hip_yaw_joint" lower="${-pi*0.5}" upper="${pi*0.5}"/>
     </joint>
     <link name="left_hip_yaw_link">
@@ -37,6 +36,5 @@
       <origin xyz="0.047875 0.00 -0.05" rpy="0.0 0.0 0.0"/>
       <axis xyz="1 0 0"/>
-      <limit velocity="4.08" effort="9.9" lower="${-pi*0.5}" upper="${pi*0.5}"/>
-      <dynamics damping="0.1" friction="0.0"/>
+      <xacro:dxl_joint_props joint="left_hip_roll_joint" lower="${-pi*0.5}" upper="${pi*0.5}"/>
     </joint>
     <link name="left_hip_roll_pitch_link">
@@ -67,6 +65,5 @@
       <origin xyz="-0.0245 0.0245 0.0" rpy="0.0 0.0 0.0"/>
       <axis xyz="0 1 0"/>
-      <limit velocity="4.08" effort="9.9" lower="${-pi*0.5}" upper="${pi*0.5}"/>
-      <dynamics damping="0.1" friction="0.0"/>
+      <xacro:dxl_joint_props joint="left_front_thigh_pitch_joint" lower="${-pi*0.5}" upper="${pi*0.5}"/>
     </joint>
     <link name="left_front_thigh_pitch_link">
@@ -84,8 +81,8 @@
       </collision>
       <inertial>
-        <origin xyz="0.011621 -0.024250 -0.106919" rpy="0.00 0.00 0.00"/>
+        <origin xyz="0.011621 -0.024250 -0.106954" rpy="0.00 0.00 0.00"/>
         <mass value="0.078"/>
         <inertia
-          ixx="0.000255" ixy="0.000003" ixz="0.000004"
+          ixx="0.000255" ixy="0.000000" ixz="0.000004"
           iyy="0.000220" iyz="0.000000"
           izz="0.000043"/>
@@ -115,9 +112,9 @@
       <inertial>
         <origin xyz="-0.010643 -0.024500 -0.094743" rpy="0.00 0.00 0.00"/>
-        <mass value="0.078"/>
-        <inertia
-          ixx="0.000255" ixy="0.000000" ixz="0.000004"
-          iyy="0.000220" iyz="0.000000"
-          izz="0.000043"/>
+        <mass value="0.0667"/>
+        <inertia
+          ixx="0.000235" ixy="0.000000" ixz="0.000001"
+          iyy="0.000202" iyz="0.000000"
+          izz="0.000039"/>
       </inertial>
     </link>
@@ -127,6 +124,5 @@
       <origin xyz="0.0 0.0 -0.2" rpy="0.0 0.0 0.0"/>
       <axis xyz="0 1 0"/>
-      <limit velocity="4.08" effort="19.8" lower="${-pi*0.5}" upper="${pi*0.5}"/>
-      <dynamics damping="0.1" friction="0.0"/>
+      <xacro:dxl_joint_props joint="left_knee_pitch_joint" lower="${-pi*0.5}" upper="${pi*0.5}"/>
     </joint>
     <link name="left_knee_pitch_link">
@@ -144,10 +140,10 @@
       </collision>
       <inertial>
-        <origin xyz="-0.005325 -0.024024 -0.017387" rpy="0.00 0.00 0.00"/>
+        <origin xyz="-0.005329 -0.024028 -0.017389" rpy="0.00 0.00 0.00"/>
         <mass value="0.34"/>
         <inertia
-          ixx="0.000242" ixy="0.000000" ixz="0.000000"
-          iyy="0.000210" iyz="0.000000"
-          izz="0.000190"/>
+          ixx="0.000200" ixy="-0.000001" ixz="-0.000008"
+          iyy="0.000231" iyz="-0.000001"
+          izz="0.000179"/>
       </inertial>
     </link>
@@ -157,6 +153,5 @@
       <origin xyz="0.0 0.0 -0.04775" rpy="0.0 0.0 0.0"/>
       <axis xyz="0 1 0"/>
-      <limit velocity="4.08" effort="9.9" lower="${-pi*0.5}" upper="${pi*0.5}"/>
-      <dynamics damping="0.1" friction="0.0"/>
+      <xacro:dxl_joint_props joint="left_front_shin_pitch_joint" lower="${-pi*0.5}" upper="${pi*0.5}"/>
     </joint>
     <link name="left_front_shin_pitch_link">
@@ -174,9 +169,9 @@
       </collision>
       <inertial>
-        <origin xyz="0.012786 -0.024250 -0.104736" rpy="0.00 0.00 0.00"/>
+        <origin xyz="0.012775 -0.024250 -0.104814" rpy="0.00 0.00 0.00"/>
         <mass value="0.079"/>
         <inertia
-          ixx="0.000259" ixy="0.000000" ixz="0.000000"
-          iyy="0.000223" iyz="0.000000"
+          ixx="0.000260" ixy="0.000000" ixz="-0.000010"
+          iyy="0.000224" iyz="0.000000"
           izz="0.000043"/>
       </inertial>
@@ -205,9 +200,9 @@
       <inertial>
         <origin xyz="-0.010643 -0.024500 -0.105257" rpy="0.00 0.00 0.00"/>
-        <mass value="0.06"/>
-        <inertia
-          ixx="0.000255" ixy="0.000000" ixz="0.000004"
-          iyy="0.000220" iyz="0.000000"
-          izz="0.000043"/>
+        <mass value="0.0667"/>
+        <inertia
+          ixx="0.000235" ixy="0.000000" ixz="-0.000001"
+          iyy="0.000202" iyz="0.000000"
+          izz="0.000039"/>
       </inertial>
     </link>
@@ -217,6 +212,5 @@
       <origin xyz="0.0 0.0 -0.2" rpy="0.0 0.0 0.0"/>
       <axis xyz="0 1 0"/>
-      <limit velocity="4.08" effort="9.9" lower="${-pi*0.5}" upper="${pi*0.5}"/>
-      <dynamics damping="0.1" friction="0.0"/>
+      <xacro:dxl_joint_props joint="left_ankle_pitch_joint" lower="${-pi*0.5}" upper="${pi*0.5}"/>
     </joint>
     <link name="left_ankle_roll_pitch_link">
@@ -234,8 +228,8 @@
       </collision>
       <inertial>
-        <origin xyz="-0.044839 -0.000311 0.015111" rpy="0.0 0.0 0.0"/>
+        <origin xyz="-0.020341 -0.024809 0.015114" rpy="0.0 0.0 0.0"/>
         <mass value="0.467377"/>
         <inertia
-          ixx="0.000198" ixy="0.000003" ixz="0.000001"
+          ixx="0.000198" ixy="-0.000003" ixz="-0.000001"
           iyy="0.000406" iyz="0.000000"
           izz="0.000326"/>
@@ -247,6 +241,5 @@
       <origin xyz="0.0245 -0.02425 0.0" rpy="0.0 0.0 0.0"/>
       <axis xyz="1 0 0"/>
-      <limit velocity="4.08" effort="9.9" lower="${-pi*0.5}" upper="${pi*0.5}"/>
-      <dynamics damping="0.1" friction="0.0"/>
+      <xacro:dxl_joint_props joint="left_ankle_roll_joint" lower="${-pi*0.5}" upper="${pi*0.5}"/>
     </joint>
     <link name="left_foot_roll_link">
@@ -267,7 +260,7 @@
         <mass value="0.229"/>
         <inertia
-          ixx="0.000557" ixy="0.000003" ixz="0.000001"
-          iyy="0.000081" iyz="0.000000"
-          izz="-0.000023"/>
+          ixx="0.000081" ixy="0.000000" ixz="0.000022"
+          iyy="0.000555" iyz="0.000000"
+          izz="0.000577"/>
       </inertial>
     </link>

File: urdf/right_arm.xacro (robot description, xacro)
@@ -7,6 +7,5 @@
       <origin xyz="-0.02089 -0.1305 0.1388" rpy="0.0 0.0873 0.0"/>
       <axis xyz="0 -1 0"/>
-      <limit velocity="3.14" effort="10.6" lower="${-pi*0.9}" upper="${pi*0.9}"/>
-      <dynamics damping="0.1" friction="0.0"/>
+      <xacro:dxl_joint_props joint="right_shoulder_pitch_joint" lower="${-pi*0.9}" upper="${pi*0.9}"/>
     </joint>
     <link name="right_shoulder_pitch_link">
@@ -18,9 +17,9 @@
       </visual>
       <inertial>
-        <origin xyz="-0.000000 -0.010235 -0.004313" rpy="0.0 0.0 0.0"/>
+        <origin xyz="0.000000 -0.010235 -0.004313" rpy="0.0 0.0 0.0"/>
         <mass value="0.044923"/>
         <inertia
           ixx="0.000013" ixy="0.000000" ixz="0.000000"
-          iyy="0.000027" iyz="0.000003"
+          iyy="0.000027" iyz="-0.000003"
           izz="0.000025"/>
       </inertial>
@@ -31,6 +30,5 @@
       <origin xyz="0.0245 -0.030017 -0.022" rpy="0.0 0.0 0.0"/>
       <axis xyz="-1 0 0"/>
-      <limit velocity="3.14" effort="10.6" lower="${-pi*0.5}" upper="${pi*0.5}"/>
-      <dynamics damping="0.1" friction="0.0"/>
+      <xacro:dxl_joint_props joint="right_shoulder_roll_joint" lower="${-pi*0.5}" upper="${pi*0.5}"/>
     </joint>
     <link name="right_shoulder_roll_link">
@@ -51,5 +49,5 @@
         <mass value="0.389041"/>
         <inertia
-          ixx="0.000698" ixy="0.000079" ixz="0.000000"
+          ixx="0.000698" ixy="-0.000079" ixz="0.000000"
           iyy="0.000117" iyz="0.000000"
           izz="0.000753"/>
@@ -61,6 +59,5 @@
       <origin xyz="-0.0245 -0.118 0.000" rpy="${-pi*0.5} 0.0 0.0"/>
       <axis xyz="0 0 1"/>
-      <limit velocity="4.82" effort="4.1" lower="${-pi*0.9}" upper="${pi*0.9}"/>
-      <dynamics damping="0.1" friction="0.0"/>
+      <xacro:dxl_joint_props joint="right_elbow_yaw_joint" lower="${-pi*0.9}" upper="${pi*0.9}"/>
     </joint>
     <link name="right_elbow_yaw_link">
@@ -72,10 +69,10 @@
       </visual>
       <inertial>
-        <origin xyz="0.003756 -0.032656 0.000000" rpy="0.0 0.0 0.0"/>
+        <origin xyz="0.003756 0.000000 -0.032656" rpy="0.0 0.0 0.0"/>
         <mass value="0.051730"/>
         <inertia
-          ixx="0.000036" ixy="-0.000005" ixz="0.000000"
-          iyy="0.000028" iyz="0.000000"
-          izz="0.000025"/>
+          ixx="0.000036" ixy="0.000000" ixz="0.000005"
+          iyy="0.000025" iyz="0.000000"
+          izz="0.000028"/>
       </inertial>
     </link>
@@ -85,6 +82,5 @@
       <origin xyz="0.022 -0.0245 -0.06" rpy="0.0 0.0 0.0"/>
       <axis xyz="0 1 0"/>
-      <limit velocity="3.14" effort="10.6" lower="${-pi*0.5}" upper="${pi*0.5}"/>
-      <dynamics damping="0.1" friction="0.0"/>
+      <xacro:dxl_joint_props joint="right_elbow_pitch_joint" lower="${-pi*0.5}" upper="${pi*0.5}"/>
     </joint>
     <link name="right_elbow_pitch_link">
@@ -102,10 +98,10 @@
       </collision>
       <inertial>
-        <origin xyz="0.000000 -0.018081 -0.023869" rpy="0.0 0.0 0.0"/>
+        <origin xyz="0.000000 0.023869 -0.018081" rpy="0.0 0.0 0.0"/>
         <mass value="0.246669"/>
         <inertia
           ixx="0.000135" ixy="0.000000" ixz="0.000000"
-          iyy="0.000064" iyz="0.000001"
-          izz="0.000121"/>
+          iyy="0.000121" iyz="0.000001"
+          izz="0.000064"/>
       </inertial>
     </link>
@@ -129,10 +125,10 @@
       </collision>
       <inertial>
-        <origin xyz="-0.000002 -0.043774 0.003217" rpy="0.0 0.0 0.0"/>
+        <origin xyz="-0.000002 -0.003217 -0.043774" rpy="0.0 0.0 0.0"/>
         <mass value="0.216195"/>
         <inertia
           ixx="0.000183" ixy="0.000000" ixz="0.000000"
-          iyy="0.000104" iyz="-0.000015"
-          izz="0.000191"/>
+          iyy="0.000191" iyz="-0.000015"
+          izz="0.000104"/>
       </inertial>
     </link>

File: urdf/right_leg.xacro (robot description, xacro)
@@ -7,6 +7,5 @@
       <origin xyz="0.0 -0.055 0.0" rpy="0.0 0.0 0.0"/>
       <axis xyz="0 0 1"/>
-      <limit velocity="4.82" effort="4.1" lower="${-pi*0.5}" upper="${pi*0.5}"/>
-      <dynamics damping="0.1" friction="0.0"/>
+      <xacro:dxl_joint_props joint="right_hip_yaw_joint" lower="${-pi*0.5}" upper="${pi*0.5}"/>
     </joint>
     <link name="right_hip_yaw_link">
@@ -37,6 +36,5 @@
       <origin xyz="0.047875 0.0 -0.05" rpy="0.0 0.0 0.0"/>
       <axis xyz="1 0 0"/>
-      <limit velocity="4.08" effort="9.9" lower="${-pi*0.5}" upper="${pi*0.5}"/>
-      <dynamics damping="0.1" friction="0.0"/>
+      <xacro:dxl_joint_props joint="right_hip_roll_joint" lower="${-pi*0.5}" upper="${pi*0.5}"/>
     </joint>
     <link name="right_hip_roll_pitch_link">
@@ -67,6 +65,5 @@
       <origin xyz="-0.0245 0.0245 0.0" rpy="0.0 0.0 0.0"/>
       <axis xyz="0 1 0"/>
-      <limit velocity="4.08" effort="19.8" lower="${-pi*0.5}" upper="${pi*0.5}"/>
-      <dynamics damping="0.1" friction="0.0"/>
+      <xacro:dxl_joint_props joint="right_front_thigh_pitch_joint" lower="${-pi*0.5}" upper="${pi*0.5}"/>
     </joint>
     <link name="right_front_thigh_pitch_link">
@@ -84,8 +81,8 @@
       </collision>
       <inertial>
-        <origin xyz="0.011621 -0.024250 -0.106919" rpy="0.00 0.00 0.00"/>
+        <origin xyz="0.011621 -0.024250 -0.106954" rpy="0.00 0.00 0.00"/>
         <mass value="0.078"/>
         <inertia
-          ixx="0.000255" ixy="0.000003" ixz="0.000004"
+          ixx="0.000255" ixy="0.000000" ixz="0.000004"
           iyy="0.000220" iyz="0.000000"
           izz="0.000043"/>
@@ -115,9 +112,9 @@
       <inertial>
         <origin xyz="-0.010643 -0.024500 -0.094743" rpy="0.00 0.00 0.00"/>
-        <mass value="0.06"/>
-        <inertia
-          ixx="0.000255" ixy="0.000000" ixz="0.000004"
-          iyy="0.000220" iyz="0.000000"
-          izz="0.000043"/>
+        <mass value="0.0667"/>
+        <inertia
+          ixx="0.000235" ixy="0.000000" ixz="0.000001"
+          iyy="0.000202" iyz="0.000000"
+          izz="0.000039"/>
       </inertial>
     </link>
@@ -127,6 +124,5 @@
       <origin xyz="0.0 0.0 -0.2" rpy="0.0 0.0 0.0"/>
       <axis xyz="0 1 0"/>
-      <limit velocity="4.08" effort="19.8" lower="${-pi*0.5}" upper="${pi*0.5}"/>
-      <dynamics damping="0.1" friction="0.0"/>
+      <xacro:dxl_joint_props joint="right_knee_pitch_joint" lower="${-pi*0.5}" upper="${pi*0.5}"/>
     </joint>
     <link name="right_knee_pitch_link">
@@ -144,10 +140,10 @@
       </collision>
       <inertial>
-        <origin xyz="-0.005325 -0.024024 -0.017387" rpy="0.00 0.00 0.00"/>
+        <origin xyz="-0.005329 -0.024028 -0.017389" rpy="0.00 0.00 0.00"/>
         <mass value="0.34"/>
         <inertia
-          ixx="0.000242" ixy="0.000000" ixz="0.000000"
-          iyy="0.000210" iyz="0.000000"
-          izz="0.000190"/>
+          ixx="0.000200" ixy="-0.000001" ixz="-0.000008"
+          iyy="0.000231" iyz="-0.000001"
+          izz="0.000179"/>
       </inertial>
     </link>
@@ -157,6 +153,5 @@
       <origin xyz="0.0 0.0 -0.04775" rpy="0.0 0.0 0.0"/>
       <axis xyz="0 1 0"/>
-      <limit velocity="4.08" effort="9.9" lower="${-pi*0.5}" upper="${pi*0.5}"/>
-      <dynamics damping="0.1" friction="0.0"/>
+      <xacro:dxl_joint_props joint="right_front_shin_pitch_joint" lower="${-pi*0.5}" upper="${pi*0.5}"/>
     </joint>
     <link name="right_front_shin_pitch_link">
@@ -174,9 +169,9 @@
       </collision>
       <inertial>
-        <origin xyz="0.012786 -0.024250 -0.104736" rpy="0.00 0.00 0.00"/>
+        <origin xyz="0.012775 -0.024250 -0.104814" rpy="0.00 0.00 0.00"/>
         <mass value="0.079"/>
         <inertia
-          ixx="0.000259" ixy="0.000000" ixz="0.000000"
-          iyy="0.000223" iyz="0.000000"
+          ixx="0.000260" ixy="0.000000" ixz="-0.000010"
+          iyy="0.000224" iyz="0.000000"
           izz="0.000043"/>
       </inertial>
@@ -205,9 +200,9 @@
       <inertial>
         <origin xyz="-0.010643 -0.024500 -0.105257" rpy="0.00 0.00 0.00"/>
-        <mass value="0.06"/>
-        <inertia
-          ixx="0.000255" ixy="0.000000" ixz="0.000004"
-          iyy="0.000220" iyz="0.000000"
-          izz="0.000043"/>
+        <mass value="0.0667"/>
+        <inertia
+          ixx="0.000235" ixy="0.000000" ixz="-0.000001"
+          iyy="0.000202" iyz="0.000000"
+          izz="0.000039"/>
       </inertial>
     </link>
@@ -217,6 +212,5 @@
       <origin xyz="0.0 0.0 -0.2" rpy="0.0 0.0 0.0"/>
       <axis xyz="0 1 0"/>
-      <limit velocity="4.08" effort="9.9" lower="${-pi*0.5}" upper="${pi*0.5}"/>
-      <dynamics damping="0.1" friction="0.0"/>
+      <xacro:dxl_joint_props joint="right_ankle_pitch_joint" lower="${-pi*0.5}" upper="${pi*0.5}"/>
     </joint>
     <link name="right_ankle_roll_pitch_link">
@@ -234,8 +228,8 @@
       </collision>
       <inertial>
-        <origin xyz="-0.044839 -0.000311 0.015111" rpy="0.0 0.0 0.0"/>
+        <origin xyz="-0.020341 -0.024809 0.015114" rpy="0.0 0.0 0.0"/>
         <mass value="0.467377"/>
         <inertia
-          ixx="0.000198" ixy="0.000003" ixz="0.000001"
+          ixx="0.000198" ixy="-0.000003" ixz="-0.000001"
           iyy="0.000406" iyz="0.000000"
           izz="0.000326"/>
@@ -247,6 +241,5 @@
       <origin xyz="0.0245 -0.02425 0.0" rpy="0.0 0.0 0.0"/>
       <axis xyz="1 0 0"/>
-      <limit velocity="4.08" effort="9.9" lower="${-pi*0.5}" upper="${pi*0.5}"/>
-      <dynamics damping="0.1" friction="0.0"/>
+      <xacro:dxl_joint_props joint="right_ankle_roll_joint" lower="${-pi*0.5}" upper="${pi*0.5}"/>
     </joint>
     <link name="right_foot_roll_link">
@@ -267,7 +260,7 @@
         <mass value="0.229"/>
         <inertia
-          ixx="0.000557" ixy="0.000003" ixz="0.000001"
-          iyy="0.000081" iyz="0.000000"
-          izz="-0.000023"/>
+          ixx="0.000081" ixy="0.000000" ixz="0.000022"
+          iyy="0.000555" iyz="0.000000"
+          izz="0.000577"/>
       </inertial>
     </link>
