Commit message: Fix link inertials and add DYNAMIXEL actuator config
Inertials (verified against mesh-derived COM/inertia for all links):
- foot: tensor entries were misplaced (negative izz, not positive-definite)
- ankle_roll_pitch: COM missing the visual origin offset
- back_thigh/back_shin: inconsistent copied mass/inertia; mass from Al density
- elbow_yaw/elbow_pitch/gripper: CAD values re-expressed in the link frame
  (visuals are rotated +-90 deg; COM was off by 42-66 mm)
- lower_body/upper_body/shoulder/head: products of inertia sign flipped to
  URDF convention; lower_body COM missing visual z offset
- knee/front_thigh/front_shin: replaced hand-entered tensors with mesh values

Actuators:
- config/actuators.yaml: single source for XH540-W270, XM540-W270,
  XM430-W350 specs at 14.8 V, joint-to-servo mapping (dual servos on hip
  pitch and knee), armature/friction priors transferred from BAM MX-series
  identifications, and BAM identification priors
- urdf/actuators.xacro: generates joint <limit>/<dynamics> from the yaml
- hip_yaw now uses XM540-W270 limits (was XM430 values)
- left_front_thigh effort fixed to dual-servo value
- Install config/ in setup.py; regenerate robinion2.urdf

File: urdf/robinion2.urdf (robot description, URDF)
Before this commit: robot robinion, 35 links, 34 joints
Links:
- link left_back_shin_pitch_link: mass 0.06 -> 0.0667
- link left_back_thigh_pitch_link: mass 0.078 -> 0.0667
- link right_back_shin_pitch_link: mass 0.06 -> 0.0667
- link right_back_thigh_pitch_link: mass 0.06 -> 0.0667
Joints:
- joint head_pitch_joint: limit lower=-1.5707963267948966 upper=1.5707963267948966 effort=4.1 velocity=4.82 -> lower=-1.5707963267948966 upper=1.5707963267948966 effort=4.8 velocity=5.969
- joint head_yaw_joint: limit lower=-1.5707963267948966 upper=1.5707963267948966 effort=4.1 velocity=4.82 -> lower=-1.5707963267948966 upper=1.5707963267948966 effort=4.8 velocity=5.969
- joint left_ankle_pitch_joint: limit lower=-1.5707963267948966 upper=1.5707963267948966 effort=9.9 velocity=4.08 -> lower=-1.5707963267948966 upper=1.5707963267948966 effort=11.7 velocity=4.817
- joint left_ankle_roll_joint: limit lower=-1.5707963267948966 upper=1.5707963267948966 effort=9.9 velocity=4.08 -> lower=-1.5707963267948966 upper=1.5707963267948966 effort=11.7 velocity=4.817
- joint left_elbow_pitch_joint: limit lower=-1.5707963267948966 upper=1.5707963267948966 effort=10.6 velocity=3.14 -> lower=-1.5707963267948966 upper=1.5707963267948966 effort=12.9 velocity=3.875
- joint left_elbow_yaw_joint: limit lower=-2.827433388230814 upper=2.827433388230814 effort=4.1 velocity=4.82 -> lower=-2.827433388230814 upper=2.827433388230814 effort=4.8 velocity=5.969
- joint left_front_shin_pitch_joint: limit lower=-1.5707963267948966 upper=1.5707963267948966 effort=9.9 velocity=4.08 -> lower=-1.5707963267948966 upper=1.5707963267948966 effort=11.7 velocity=4.817
- joint left_front_thigh_pitch_joint: limit lower=-1.5707963267948966 upper=1.5707963267948966 effort=9.9 velocity=4.08 -> lower=-1.5707963267948966 upper=1.5707963267948966 effort=23.4 velocity=4.817
- joint left_hip_roll_joint: limit lower=-1.5707963267948966 upper=1.5707963267948966 effort=9.9 velocity=4.08 -> lower=-1.5707963267948966 upper=1.5707963267948966 effort=11.7 velocity=4.817
- joint left_hip_yaw_joint: limit lower=-1.5707963267948966 upper=1.5707963267948966 effort=4.1 velocity=4.82 -> lower=-1.5707963267948966 upper=1.5707963267948966 effort=12.9 velocity=3.875
- joint left_knee_pitch_joint: limit lower=-1.5707963267948966 upper=1.5707963267948966 effort=19.8 velocity=4.08 -> lower=-1.5707963267948966 upper=1.5707963267948966 effort=23.4 velocity=4.817
- joint left_shoulder_pitch_joint: limit lower=-2.827433388230814 upper=2.827433388230814 effort=10.6 velocity=3.14 -> lower=-2.827433388230814 upper=2.827433388230814 effort=12.9 velocity=3.875
- joint left_shoulder_roll_joint: limit lower=-1.5707963267948966 upper=1.5707963267948966 effort=10.6 velocity=3.14 -> lower=-1.5707963267948966 upper=1.5707963267948966 effort=12.9 velocity=3.875
- joint right_ankle_pitch_joint: limit lower=-1.5707963267948966 upper=1.5707963267948966 effort=9.9 velocity=4.08 -> lower=-1.5707963267948966 upper=1.5707963267948966 effort=11.7 velocity=4.817
- joint right_ankle_roll_joint: limit lower=-1.5707963267948966 upper=1.5707963267948966 effort=9.9 velocity=4.08 -> lower=-1.5707963267948966 upper=1.5707963267948966 effort=11.7 velocity=4.817
- joint right_elbow_pitch_joint: limit lower=-1.5707963267948966 upper=1.5707963267948966 effort=10.6 velocity=3.14 -> lower=-1.5707963267948966 upper=1.5707963267948966 effort=12.9 velocity=3.875
- joint right_elbow_yaw_joint: limit lower=-2.827433388230814 upper=2.827433388230814 effort=4.1 velocity=4.82 -> lower=-2.827433388230814 upper=2.827433388230814 effort=4.8 velocity=5.969
- joint right_front_shin_pitch_joint: limit lower=-1.5707963267948966 upper=1.5707963267948966 effort=9.9 velocity=4.08 -> lower=-1.5707963267948966 upper=1.5707963267948966 effort=11.7 velocity=4.817
- joint right_front_thigh_pitch_joint: limit lower=-1.5707963267948966 upper=1.5707963267948966 effort=19.8 velocity=4.08 -> lower=-1.5707963267948966 upper=1.5707963267948966 effort=23.4 velocity=4.817
- joint right_hip_roll_joint: limit lower=-1.5707963267948966 upper=1.5707963267948966 effort=9.9 velocity=4.08 -> lower=-1.5707963267948966 upper=1.5707963267948966 effort=11.7 velocity=4.817
- joint right_hip_yaw_joint: limit lower=-1.5707963267948966 upper=1.5707963267948966 effort=4.1 velocity=4.82 -> lower=-1.5707963267948966 upper=1.5707963267948966 effort=12.9 velocity=3.875
- joint right_knee_pitch_joint: limit lower=-1.5707963267948966 upper=1.5707963267948966 effort=19.8 velocity=4.08 -> lower=-1.5707963267948966 upper=1.5707963267948966 effort=23.4 velocity=4.817
- joint right_shoulder_pitch_joint: limit lower=-2.827433388230814 upper=2.827433388230814 effort=10.6 velocity=3.14 -> lower=-2.827433388230814 upper=2.827433388230814 effort=12.9 velocity=3.875
- joint right_shoulder_roll_joint: limit lower=-1.5707963267948966 upper=1.5707963267948966 effort=10.6 velocity=3.14 -> lower=-1.5707963267948966 upper=1.5707963267948966 effort=12.9 velocity=3.875
- joint torso_pitch_joint: limit lower=-0.52 upper=1.5707963267948966 effort=10.6 velocity=3.14 -> lower=-0.52 upper=1.5707963267948966 effort=12.9 velocity=3.875

File: urdf/robinion2.xacro (robot description, xacro)
@@ -1,4 +1,5 @@
 <?xml version="1.0"?>
 <robot name="robinion" xmlns:xacro="http://www.ros.org/wiki/xacro">
+  <xacro:include filename="$(find robinion_description)/urdf/actuators.xacro"/>
   <xacro:include filename="$(find robinion_description)/urdf/body.xacro"/>
   <xacro:include filename="$(find robinion_description)/urdf/head.xacro"/>
